Commit message: description: add rviz debugging launch

File: rarog_description/urdf/rarog.urdf.xacro (robot description, xacro)
@@ -2,4 +2,5 @@
 <robot xmlns:xacro="http://www.ros.org/wiki/xacro"
   name="rarog">
+  <xacro:property name="pi" value="3.141592653589793" />
   <link name="base_link">
     <!-- Robot base link
@@ -12,5 +13,5 @@
     </inertial> -->
     <visual>
-      <origin xyz="0 0 0" rpy="0 0 0" />
+      <origin xyz="0 0 10" rpy="${pi} 0 0" />
       <geometry>
         <!-- XXX TODO Rarog uses Skywalker V6 1900, need to find right model -->

Commit message: description: fix collada format. Only meters allowed!

File: rarog_description/urdf/rarog.urdf.xacro (robot description, xacro)
@@ -16,5 +16,5 @@
       <geometry>
         <!-- XXX TODO Rarog uses Skywalker V6 1900, need to find right model -->
-        <mesh filename="package://rarog_description/meshes/skywalker_2013.dae"/>
+        <mesh filename="package://rarog_description/meshes/t.dae"/>
       </geometry>
       <material name="red">

Commit message: description: rviz now show me a model

File: rarog_description/urdf/rarog.urdf.xacro (robot description, xacro)
@@ -13,10 +13,10 @@
     </inertial> -->
     <visual>
-      <origin xyz="0 0 10" rpy="${pi} 0 0" />
+      <origin xyz="0 0 -0.13" rpy="${pi} 0 0" />
       <geometry>
         <!-- XXX TODO Rarog uses Skywalker V6 1900, need to find right model -->
-        <mesh filename="package://rarog_description/meshes/t.dae"/>
+        <mesh filename="package://rarog_description/meshes/skywalker_2013.dae"/>
       </geometry>
-      <material name="red">
+      <material name="red"> <!-- GOES FASTA! -->
         <color rgba=".8 0 0 1" />
       </material>
@@ -25,4 +25,12 @@
   <link name="fcu">
     <!-- FCU frame (mavros uses this link for most topics) -->
+    <visual>
+      <geometry>
+        <box size=".085 .052 .02" />
+      </geometry>
+      <material name="dark-grey">
+        <color rgba=".2 .2 .2 1" />
+      </material>
+    </visual>
   </link>
   <joint name="base_to_fcu" type="fixed">
@@ -32,5 +40,5 @@
          +5 cm X, -3 cm Y from CoG (wing lower plane)
          -->
-    <origin xyz="0.005 0 -0.003" rpy="0 0 0" />
+    <origin xyz="0.05 0 -0.03" rpy="0 0 0" />
   </joint>
   <!-- vim: set ts=2 sw=2 et : -->

Commit message: description: add ailerons to urdf

File: rarog_description/urdf/rarog.urdf.xacro (robot description, xacro)
@@ -1,6 +1,20 @@
-<?xml version="1.0"?>
+<?xml version="1.0" encoding="UTF-8"?>
 <robot xmlns:xacro="http://www.ros.org/wiki/xacro"
   name="rarog">
-  <xacro:property name="pi" value="3.141592653589793" />
+  <!--
+    RAROG UAV
+    =========
+    It is my very own drone for reserch navigation planning and filming.
+    Maybe that package may help you to define your UAV.
+    Airframe: Skywalker V6 1900
+    FCU: Pixhawk with PX4 firmware
+    OBC: Raspberry Pi 2 with Ubuntu 14.04 armhf
+    Weight: ~2 kg
+    ~~~~ Vladimir Ermakov <vooon341@gmail.com>
+       -->
+  <!-- NOTE: xacro dont care about encoding, non ascii cause an error -->
+  <!-- in Jade math.pi predefined -->
+  <xacro:property name="add_control_surfaces" value="true" />
+  <xacro:property name="kgcm_to_nm" value="0.0980665" />
   <link name="base_link">
     <!-- Robot base link
@@ -42,4 +56,40 @@
     <origin xyz="0.05 0 -0.03" rpy="0 0 0" />
   </joint>
+  <xacro:macro name="aileron" params="link *material *origin">
+    <link name="${link}">
+      <visual>
+        <geometry>
+          <!-- Aileron trapeze: 6 - 24.5 - 5 cm -->
+          <box size=".055 .245 .005" />
+        </geometry>
+        <xacro:insert_block name="material" />
+        <origin xyz="${-0.055/2} 0 0" rpy="0 0 0" />
+      </visual>
+    </link>
+    <joint name="base_to_${link}" type="revolute">
+      <parent link="base_link" />
+      <child link="${link}" />
+      <xacro:insert_block name="origin" />
+      <axis xyz="0 1 0" />
+      <!-- Lets say 30 deg, servo: 1.5 kg*cm (6 volt), 60 deg in 0.10 sec -->
+      <limit lower="${radians(-30)}" upper="${radians(30)}" effort="${1.5 * kgcm_to_nm}" velocity="${radians(60. / 0.10)}" />
+    </joint>
+  </xacro:macro>
+  <xacro:if value="${add_control_surfaces}">
+    <!-- <joint name="aileron_link" /> -->
+    <!-- aileron location: 51 cm Y to 6-cm side, -5 cm on X -->
+    <xacro:aileron link="aileron_left">
+      <material name="red">
+        <color rgba=".9 0 0 1" />
+      </material>
+      <origin xyz="-0.05 ${.51 + .245/2} .02" rpy="0 0 0" />
+    </xacro:aileron>
+    <xacro:aileron link="aileron_right">
+      <material name="green">
+        <color rgba="0 .9 0 1" />
+      </material>
+      <origin xyz="-0.05 ${-(.51 + .245/2)} .02" rpy="0 0 0" />
+    </xacro:aileron>
+  </xacro:if>
   <!-- vim: set ts=2 sw=2 et : -->
 </robot>

Commit message: description: single joint for aileron (l/r are mimic)

File: rarog_description/urdf/rarog.urdf.xacro (robot description, xacro)
@@ -56,5 +56,9 @@
     <origin xyz="0.05 0 -0.03" rpy="0 0 0" />
   </joint>
-  <xacro:macro name="aileron" params="link *material *origin">
+  <xacro:macro name="aileron_servo_limit">
+      <!-- Lets say 30 deg, servo: 1.5 kg*cm (6 volt), 60 deg in 0.10 sec -->
+      <limit lower="${radians(-30)}" upper="${radians(30)}" effort="${1.5 * kgcm_to_nm}" velocity="${radians(60. / 0.10)}" />
+  </xacro:macro>
+  <xacro:macro name="aileron" params="link *material *origin *mimic">
     <link name="${link}">
       <visual>
@@ -72,11 +76,18 @@
       <xacro:insert_block name="origin" />
       <axis xyz="0 1 0" />
-      <!-- Lets say 30 deg, servo: 1.5 kg*cm (6 volt), 60 deg in 0.10 sec -->
-      <limit lower="${radians(-30)}" upper="${radians(30)}" effort="${1.5 * kgcm_to_nm}" velocity="${radians(60. / 0.10)}" />
+      <xacro:aileron_servo_limit />
+      <xacro:insert_block name="mimic" />
     </joint>
   </xacro:macro>
   <xacro:if value="${add_control_surfaces}">
-    <!-- <joint name="aileron_link" /> -->
+    <!-- conventional ailerons controlled by one axis -->
+    <link name="aileron_link" />
+    <joint name="base_to_aileron" type="revolute">
+      <parent link="base_link" />
+      <child link="aileron_link" />
+      <xacro:aileron_servo_limit />
+    </joint>
     <!-- aileron location: 51 cm Y to 6-cm side, -5 cm on X -->
+    <!-- TODO check mimic tags -->
     <xacro:aileron link="aileron_left">
       <material name="red">
@@ -84,4 +95,5 @@
       </material>
       <origin xyz="-0.05 ${.51 + .245/2} .02" rpy="0 0 0" />
+      <mimic joint="base_to_aileron" multiplier="-1" />
     </xacro:aileron>
     <xacro:aileron link="aileron_right">
@@ -90,5 +102,10 @@
       </material>
       <origin xyz="-0.05 ${-(.51 + .245/2)} .02" rpy="0 0 0" />
+      <mimic joint="base_to_aileron" multiplier="1" />
     </xacro:aileron>
+    <joint name="elevator_link">
+      <visual>
+      </visual>
+    </joint>
   </xacro:if>
   <!-- vim: set ts=2 sw=2 et : -->

Commit message: description: add evelator and rudder to urdf

File: rarog_description/urdf/rarog.urdf.xacro (robot description, xacro)
@@ -18,7 +18,5 @@
   <xacro:property name="kgcm_to_nm" value="0.0980665" />
   <link name="base_link">
-    <!-- Robot base link
-         TODO: Ensure that it connected to CoG
-         -->
+    <!-- Robot base link: near CoG -->
     <!-- TODO <inertial>
       <mass value="2.0" />
@@ -52,9 +50,9 @@
     <child link="fcu" />
     <!-- FCU located under wing, on symmetry line,
-         +5 cm X, -3 cm Y from CoG (wing lower plane)
+         +5 cm X, -3 cm Y from base_link
          -->
     <origin xyz="0.05 0 -0.03" rpy="0 0 0" />
   </joint>
-  <xacro:macro name="aileron_servo_limit">
+  <xacro:macro name="common_servo_limit">
       <!-- Lets say 30 deg, servo: 1.5 kg*cm (6 volt), 60 deg in 0.10 sec -->
       <limit lower="${radians(-30)}" upper="${radians(30)}" effort="${1.5 * kgcm_to_nm}" velocity="${radians(60. / 0.10)}" />
@@ -71,10 +69,10 @@
       </visual>
     </link>
-    <joint name="base_to_${link}" type="revolute">
+    <joint name="${link}" type="revolute">
       <parent link="base_link" />
       <child link="${link}" />
       <xacro:insert_block name="origin" />
       <axis xyz="0 1 0" />
-      <xacro:aileron_servo_limit />
+      <xacro:common_servo_limit />
       <xacro:insert_block name="mimic" />
     </joint>
@@ -83,11 +81,10 @@
     <!-- conventional ailerons controlled by one axis -->
     <link name="aileron_link" />
-    <joint name="base_to_aileron" type="revolute">
+    <joint name="aileron" type="revolute">
       <parent link="base_link" />
       <child link="aileron_link" />
-      <xacro:aileron_servo_limit />
+      <xacro:common_servo_limit />
     </joint>
     <!-- aileron location: 51 cm Y to 6-cm side, -5 cm on X -->
-    <!-- TODO check mimic tags -->
     <xacro:aileron link="aileron_left">
       <material name="red">
@@ -95,5 +92,5 @@
       </material>
       <origin xyz="-0.05 ${.51 + .245/2} .02" rpy="0 0 0" />
-      <mimic joint="base_to_aileron" multiplier="-1" />
+      <mimic joint="aileron" multiplier="-1" />
     </xacro:aileron>
     <xacro:aileron link="aileron_right">
@@ -102,9 +99,43 @@
       </material>
       <origin xyz="-0.05 ${-(.51 + .245/2)} .02" rpy="0 0 0" />
-      <mimic joint="base_to_aileron" multiplier="1" />
+      <mimic joint="aileron" multiplier="1" />
     </xacro:aileron>
-    <joint name="elevator_link">
+    <!-- Elevator (T-tail) -->
+    <link name="elevator_link">
       <visual>
+        <geometry>
+          <box size=".035 .54 .005" />
+        </geometry>
+        <material name="blue">
+          <color rgba="0 0 .9 1" />
+        </material>
+        <origin xyz="${-0.035/2} 0 0" rpy="0 0 0" />
       </visual>
+    </link>
+    <joint name="elevator" type="revolute">
+      <parent link="base_link" />
+      <child link="elevator_link" />
+      <origin xyz="-0.75 0 .07" rpy="0 0 0" />
+      <axis xyz="0 1 0" />
+      <xacro:common_servo_limit />
+    </joint>
+    <!-- Rudder (T-tail) -->
+    <link name="rudder_link">
+      <visual>
+        <geometry>
+          <box size=".07 .005 .165" />
+        </geometry>
+        <material name="yellow">
+          <color rgba=".9 .9 0 1" />
+        </material>
+        <origin xyz="${-0.07/2} 0 0" rpy="0 0 0" />
+      </visual>
+    </link>
+    <joint name="rudder" type="revolute">
+      <parent link="base_link" />
+      <child link="rudder_link" />
+      <origin xyz="-0.71 0 -0.05" rpy="0 0 0" />
+      <axis xyz="0 0 1" />
+      <xacro:common_servo_limit />
     </joint>
   </xacro:if>
